File: mbavr-1t/mbavr-1t.brd (EAGLE design)
At the start: 27 x 27.9 mm, 9 parts

Commit message: Update R2 value.
Parts:
- R1: value 50k -> 10k
- R2: value 1k2 -> 560R
Changed lines of the file:
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@@
 <attribute name="VALUE" x="35.23" y="64.965" size="1.016" layer="28" rot="MR180"/>
 </element>
-<element name="R1" library="resistor" package="R1206" value="50k" x="19.685" y="54.61" smashed="yes" rot="MR0">
+<element name="R1" library="resistor" package="R1206" value="10k" x="19.685" y="54.61" smashed="yes" rot="MR0">
 <attribute name="NAME" x="24.765" y="53.975" size="1.27" layer="26" rot="MR0"/>
 <attribute name="VALUE" x="20.955" y="52.07" size="1.27" layer="28" rot="MR0"/>
 </element>
-<element name="R2" library="resistor" package="R1206" value="1k2" x="29.21" y="63.5" smashed="yes" rot="R90">
+<element name="R2" library="resistor" package="R1206" value="560R" x="29.21" y="63.5" smashed="yes" rot="R90">
 <attribute name="NAME" x="31.75" y="62.23" size="1.27" layer="25" rot="R90"/>
 <attribute name="VALUE" x="31.75" y="62.23" size="1.27" layer="27" rot="R90"/>
